File: hardware/m2-2280/thinkmoth-nvme-m2-2280.kicad_pcb (KiCad board)
At the start: 2 copper layers, 50.7 x 97 mm, 18 parts, among them J2 ExpressCard, J3 MDT180M03001, U1 GL823K-HCY04

Commit message: updates
Parts:
- added ?: , , F.Cu at (63.0, 117.3)
- added H4: MOUNTING SCREW, MountingHole:MountingHole_2.2mm_M2, F.Cu at (63.0, 117.3)
- added H5: MOUNTING SCREW, MountingHole:MountingHole_2.2mm_M2, F.Cu at (89.1, 117.3)
- added R3: 0r, Resistor_SMD:R_0402_1005Metric, F.Cu at (62.9, 65.0)
- added R4: 0r, Resistor_SMD:R_0402_1005Metric, F.Cu at (62.3, 64.3)
- Card1: moved to B.Cu
- R1, R2: value 680r -> 4k
- moved H3 63.5 mm to (88.8, 77.8)
- moved H4 45.5 mm to (62.9, 145.2)
- moved U1 24.8 mm to (70.4, 61.1)
- moved Card1 24.5 mm to (83.0, 62.9), turned to 180 degrees
- moved C4 23.2 mm to (70.5, 65.2)
- moved R2 20.1 mm to (90.1, 150.2)
- moved D2 19.5 mm to (89.1, 152.0)
- moved H5 19.4 mm to (89.0, 145.2)
- moved H1 18.0 mm to (75.6, 150.8), turned to 0 degrees
- moved C2 12.4 mm to (81.0, 64.4)
- moved C1 11.7 mm to (81.0, 63.5)
- moved J3 9.23 mm to (75.9, 68.0), turned to 0 degrees
- moved D1 8.74 mm to (62.7, 152.0)
- moved R1 8.02 mm to (61.2, 150.2)
Connections:
- R1 pad 2: PCIe_LED -> PCIe_LED_S
- R2 pad 2: SD_LED -> SD_LED_S
Routing:
- net SD_LED_S: track 0.00 -> 119.6 mm, vias 0 -> 2
- net PCIe_LED_S: track 0.00 -> 86.6 mm, vias 0 -> 2
- net 3V3: track 0.26 -> 28.0 mm, vias 0 -> 4
- net CLKREQ: track 0.00 -> 20.9 mm, vias 0 -> 2
- net SD_DAT1: track 0.00 -> 20.8 mm, vias 0 -> 1
- net SD_DAT2: track 0.00 -> 20.2 mm, vias 0 -> 1
- net SD_CLK: track 0.00 -> 20.2 mm, vias 0 -> 1
- net SD_DAT0: track 0.00 -> 19.7 mm, vias 0 -> 1
- net SD_DAT3: track 0.00 -> 19.6 mm, vias 0 -> 1
- net SD_CMD: track 0.00 -> 19.4 mm, vias 0 -> 1
- net PCIe_RX_P: track 0.00 -> 18.3 mm
- net PCIe_RX_N: track 0.00 -> 18.3 mm
- net SD_3V3: track 0.00 -> 18.1 mm, vias 0 -> 1
- net PERST: track 1.61 -> 19.7 mm, vias 1 -> 2
- net PCIe_CLK_P: track 0.00 -> 18.0 mm, vias 0 -> 2
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- added copper zone on B.Cu, net 3V3
- added copper zone on F.Cu, net 3V3
Other:
- board size 50.7 x 97 mm -> 31 x 99.5 mm
- board text added: "Extra Long M.2 2280"
- board text added: "LED Jumpers R3: PCIe R4: uSD"
- board text added: "NVMe only!!!"
- board text removed: "M.2 2242"
